File: PCB/CawBMS.kicad_sch (KiCad schematic)
At the start: 37 parts, among them CN1 SWD, CN2 I2C, CN3 SPI, CN4 USART, CN5 SWD, SW1 B3U-1000P, SW2 B3U-1000P, U1 STM32F103CBTx, U2 TCAN1044DRBRQ1, U5 CAN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

Commit message: 调整丝印 📐
Connections:
- net I2C2_SCL: now also CN2.2; no longer CN2.1
- net I2C2_SDA: now also CN2.1; no longer CN2.2
- no-connect marks 29 -> 31
Changed lines of the file:
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@@
   (no_connect (at 113.03 52.07))
   (no_connect (at 113.03 69.85))
+  (no_connect (at 132.08 148.59))
   (no_connect (at 64.77 158.75))
   (no_connect (at 77.47 166.37))
@@
   (no_connect (at 113.03 67.31))
   (no_connect (at 80.01 80.01))
+  (no_connect (at 132.08 166.37))
   (no_connect (at 133.35 182.88))
   (no_connect (at 113.03 72.39))
@@
     (effects (font (size 1.27 1.27)) (justify left bottom))
   )
-  (label "I2C2_SCL" (at 49.53 146.05 0) (fields_autoplaced)
+  (label "I2C2_SCL" (at 49.53 148.59 0) (fields_autoplaced)
     (effects (font (size 1.27 1.27)) (justify left bottom))
   )
@@
     (effects (font (size 1.27 1.27)) (justify right bottom))
   )
-  (label "I2C2_SDA" (at 49.53 148.59 0) (fields_autoplaced)
+  (label "I2C2_SDA" (at 49.53 146.05 0) (fields_autoplaced)
     (effects (font (size 1.27 1.27)) (justify left bottom))
   )
